File: hardware/kicad/m1-rf/por10-m1-rf.kicad_sch (KiCad schematic)
At the start: 4 parts, among them U1 Si4735-D60-SSOP24, X1 32.768kHz

Commit message: M1.3: move C5 inside schematic root
Parts:
- added C5: 22pF C0G, symbol Device:C
Changed lines of the file:
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@@
 		)
 	)
-  (sheet_instances
-    (path "/" (page "1"))
-  )
-)
-		(wire (pts (xy 139.7 96.52) (xy 143.51 96.52)) (stroke (width 0) (type default)))
-	(wire (pts (xy 114.3 109.22) (xy 111.76 109.22) (xy 111.76 116.84) (xy 151.13 116.84) (xy 151.13 96.52)) (stroke (width 0) (type default)))
-  (symbol
+(symbol
     (lib_id "Device:C")
     (at 143.51 100.33 0)
@@
     (instances (project "por10-m1-rf" (path "/2b0f5db7-74f4-4a9a-bfc8-7bcbf6f10a13" (reference "C5") (unit 1))))
   )
+  (sheet_instances
+    (path "/" (page "1"))
+  )
+)
+		(wire (pts (xy 139.7 96.52) (xy 143.51 96.52)) (stroke (width 0) (type default)))
+	(wire (pts (xy 114.3 109.22) (xy 111.76 109.22) (xy 111.76 116.84) (xy 151.13 116.84) (xy 151.13 96.52)) (stroke (width 0) (type default)))
   (symbol
     (lib_id "Device:C")

Commit message: M1.3: move C6 inside schematic root
Parts:
- added C6: 22pF C0G, symbol Device:C
Changed lines of the file:
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@@
     (instances (project "por10-m1-rf" (path "/2b0f5db7-74f4-4a9a-bfc8-7bcbf6f10a13" (reference "C5") (unit 1))))
   )
-  (sheet_instances
-    (path "/" (page "1"))
-  )
-)
-		(wire (pts (xy 139.7 96.52) (xy 143.51 96.52)) (stroke (width 0) (type default)))
-	(wire (pts (xy 114.3 109.22) (xy 111.76 109.22) (xy 111.76 116.84) (xy 151.13 116.84) (xy 151.13 96.52)) (stroke (width 0) (type default)))
-  (symbol
+(symbol
     (lib_id "Device:C")
     (at 151.13 100.33 0)
@@
     (instances (project "por10-m1-rf" (path "/2b0f5db7-74f4-4a9a-bfc8-7bcbf6f10a13" (reference "C6") (unit 1))))
   )
+  (sheet_instances
+    (path "/" (page "1"))
+  )
+)
+		(wire (pts (xy 139.7 96.52) (xy 143.51 96.52)) (stroke (width 0) (type default)))
+	(wire (pts (xy 114.3 109.22) (xy 111.76 109.22) (xy 111.76 116.84) (xy 151.13 116.84) (xy 151.13 96.52)) (stroke (width 0) (type default)))
   (symbol
     (lib_id "Device:C")

Commit message: M1.3: move C2 inside schematic root
Parts:
- added C2: 1nF, symbol Device:C
Changed lines of the file:
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@@
     (instances (project "por10-m1-rf" (path "/2b0f5db7-74f4-4a9a-bfc8-7bcbf6f10a13" (reference "C6") (unit 1))))
   )
-  (sheet_instances
-    (path "/" (page "1"))
-  )
-)
-		(wire (pts (xy 139.7 96.52) (xy 143.51 96.52)) (stroke (width 0) (type default)))
-	(wire (pts (xy 114.3 109.22) (xy 111.76 109.22) (xy 111.76 116.84) (xy 151.13 116.84) (xy 151.13 96.52)) (stroke (width 0) (type default)))
-  (symbol
+(symbol
     (lib_id "Device:C")
     (at 124.46 96.52 90)
@@
     (instances (project "por10-m1-rf" (path "/2b0f5db7-74f4-4a9a-bfc8-7bcbf6f10a13" (reference "C2") (unit 1))))
   )
+  (sheet_instances
+    (path "/" (page "1"))
+  )
+)
+		(wire (pts (xy 139.7 96.52) (xy 143.51 96.52)) (stroke (width 0) (type default)))
+	(wire (pts (xy 114.3 109.22) (xy 111.76 109.22) (xy 111.76 116.84) (xy 151.13 116.84) (xy 151.13 96.52)) (stroke (width 0) (type default)))
   (symbol
     (lib_id "Device:C")

Commit message: M1.3: move C3 inside schematic root
Parts:
- added C3: 0.47uF, symbol Device:C
Changed lines of the file:
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@@
     (instances (project "por10-m1-rf" (path "/2b0f5db7-74f4-4a9a-bfc8-7bcbf6f10a13" (reference "C2") (unit 1))))
   )
-  (sheet_instances
-    (path "/" (page "1"))
-  )
-)
-		(wire (pts (xy 139.7 96.52) (xy 143.51 96.52)) (stroke (width 0) (type default)))
-	(wire (pts (xy 114.3 109.22) (xy 111.76 109.22) (xy 111.76 116.84) (xy 151.13 116.84) (xy 151.13 96.52)) (stroke (width 0) (type default)))
-  (symbol
+(symbol
     (lib_id "Device:C")
     (at 124.46 106.68 90)
@@
     (instances (project "por10-m1-rf" (path "/2b0f5db7-74f4-4a9a-bfc8-7bcbf6f10a13" (reference "C3") (unit 1))))
   )
+  (sheet_instances
+    (path "/" (page "1"))
+  )
+)
+		(wire (pts (xy 139.7 96.52) (xy 143.51 96.52)) (stroke (width 0) (type default)))
+	(wire (pts (xy 114.3 109.22) (xy 111.76 109.22) (xy 111.76 116.84) (xy 151.13 116.84) (xy 151.13 96.52)) (stroke (width 0) (type default)))
   (symbol
     (lib_id "Connector:TestPoint")

Commit message: M1.3: move TP_AMI inside schematic root
Parts:
- added TP_AMI: AM_FERRITE_TEST, symbol Connector:TestPoint
Changed lines of the file:
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@@
     (instances (project "por10-m1-rf" (path "/2b0f5db7-74f4-4a9a-bfc8-7bcbf6f10a13" (reference "C3") (unit 1))))
   )
-  (sheet_instances
-    (path "/" (page "1"))
-  )
-)
-		(wire (pts (xy 139.7 96.52) (xy 143.51 96.52)) (stroke (width 0) (type default)))
-	(wire (pts (xy 114.3 109.22) (xy 111.76 109.22) (xy 111.76 116.84) (xy 151.13 116.84) (xy 151.13 96.52)) (stroke (width 0) (type default)))
-  (symbol
+(symbol
     (lib_id "Connector:TestPoint")
     (at 116.84 106.68 0)
@@
     (instances (project "por10-m1-rf" (path "/2b0f5db7-74f4-4a9a-bfc8-7bcbf6f10a13" (reference "TP_AMI") (unit 1))))
   )
+  (sheet_instances
+    (path "/" (page "1"))
+  )
+)
+		(wire (pts (xy 139.7 96.52) (xy 143.51 96.52)) (stroke (width 0) (type default)))
+	(wire (pts (xy 114.3 109.22) (xy 111.76 109.22) (xy 111.76 116.84) (xy 151.13 116.84) (xy 151.13 96.52)) (stroke (width 0) (type default)))
   (symbol
     (lib_id "Connector_Generic:Conn_01x02")

Commit message: M1.3: revert unsafe TP_AMI root move
Parts:
- removed TP_AMI: AM_FERRITE_TEST, symbol Connector:TestPoint
Changed lines of the file:
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@@
     (instances (project "por10-m1-rf" (path "/2b0f5db7-74f4-4a9a-bfc8-7bcbf6f10a13" (reference "C3") (unit 1))))
   )
-(symbol
+  (sheet_instances
+    (path "/" (page "1"))
+  )
+)(symbol
     (lib_id "Connector:TestPoint")
     (at 116.84 106.68 0)
@@
     (instances (project "por10-m1-rf" (path "/2b0f5db7-74f4-4a9a-bfc8-7bcbf6f10a13" (reference "TP_AMI") (unit 1))))
   )
-  (sheet_instances
-    (path "/" (page "1"))
-  )
-)
 		(wire (pts (xy 139.7 96.52) (xy 143.51 96.52)) (stroke (width 0) (type default)))
 	(wire (pts (xy 114.3 109.22) (xy 111.76 109.22) (xy 111.76 116.84) (xy 151.13 116.84) (xy 151.13 96.52)) (stroke (width 0) (type default)))

Commit message: M1.3: embed KiCad TestPoint library symbol
Parts:
- added TP: TestPoint
Changed lines of the file:
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@@
 (kicad_sch
-  (version 20250114)
+  		(symbol "Connector:TestPoint"
+					(pin_numbers
+						(hide yes)
+					)
+					(pin_names
+						(offset 0.762)
+						(hide yes)
+					)
+					(exclude_from_sim no)
+					(in_bom yes)
+					(on_board yes)
+					(property "Reference" "TP"
+						(at 0 6.858 0)
+						(effects
+							(font
+								(size 1.27 1.27)
+							)
+						)
+					)
+					(property "Value" "TestPoint"
+						(at 0 5.08 0)
+						(effects
+							(font
+								(size 1.27 1.27)
+							)
+						)
+					)
+					(property "Footprint" ""
+						(at 5.08 0 0)
+						(effects
+							(font
+								(size 1.27 1.27)
+							)
+							(hide yes)
+						)
+					)
+					(property "Datasheet" "~"
+						(at 5.08 0 0)
+						(effects
+							(font
+								(size 1.27 1.27)
+							)
+							(hide yes)
+						)
+					)
+					(property "Description" "test point"
+						(at 0 0 0)
+						(effects
+							(font
+								(size 1.27 1.27)
+							)
+							(hide yes)
+						)
+					)
+					(property "ki_keywords" "test point tp"
+						(at 0 0 0)
+						(effects
+							(font
+								(size 1.27 1.27)
+							)
+							(hide yes)
+						)
+					)
+					(property "ki_fp_filters" "Pin* Test*"
+						(at 0 0 0)
+						(effects
+							(font
+								(size 1.27 1.27)
+							)
+							(hide yes)
+						)
+					)
+					(symbol "TestPoint_0_1"
+						(circle
+							(center 0 3.302)
+							(radius 0.762)
+							(stroke
+								(width 0)
+								(type default)
+							)
+							(fill
+								(type none)
+							)
+						)
+					)
+					(symbol "TestPoint_1_1"
+						(pin passive line
+							(at 0 0 90)
+							(length 2.54)
+							(name "1"
+								(effects
+									(font
+										(size 1.27 1.27)
+									)
+								)
+							)
+							(number "1"
+								(effects
+									(font
+										(size 1.27 1.27)
+									)
+								)
+							)
+						)
+					)
+					(embedded_fonts no)
+				)
+(version 20250114)
   (generator "eeschema")
   (generator_version "9.0")

Commit message: M1.3: correctly embed TestPoint library symbol
Parts:
- removed TP: TestPoint
Changed lines of the file:
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@@
 (kicad_sch
-  		(symbol "Connector:TestPoint"
-					(pin_numbers
-						(hide yes)
-					)
-					(pin_names
-						(offset 0.762)
-						(hide yes)
-					)
-					(exclude_from_sim no)
-					(in_bom yes)
-					(on_board yes)
-					(property "Reference" "TP"
-						(at 0 6.858 0)
-						(effects
-							(font
-								(size 1.27 1.27)
-							)
-						)
-					)
-					(property "Value" "TestPoint"
-						(at 0 5.08 0)
-						(effects
-							(font
-								(size 1.27 1.27)
-							)
-						)
-					)
-					(property "Footprint" ""
-						(at 5.08 0 0)
-						(effects
-							(font
-								(size 1.27 1.27)
-							)
-							(hide yes)
-						)
-					)
-					(property "Datasheet" "~"
-						(at 5.08 0 0)
-						(effects
-							(font
-								(size 1.27 1.27)
-							)
-							(hide yes)
-						)
-					)
-					(property "Description" "test point"
-						(at 0 0 0)
-						(effects
-							(font
-								(size 1.27 1.27)
-							)
-							(hide yes)
-						)
-					)
-					(property "ki_keywords" "test point tp"
-						(at 0 0 0)
-						(effects
-							(font
-								(size 1.27 1.27)
-							)
-							(hide yes)
-						)
-					)
-					(property "ki_fp_filters" "Pin* Test*"
-						(at 0 0 0)
-						(effects
-							(font
-								(size 1.27 1.27)
-							)
-							(hide yes)
-						)
-					)
-					(symbol "TestPoint_0_1"
-						(circle
-							(center 0 3.302)
-							(radius 0.762)
-							(stroke
-								(width 0)
-								(type default)
-							)
-							(fill
-								(type none)
-							)
-						)
-					)
-					(symbol "TestPoint_1_1"
-						(pin passive line
-							(at 0 0 90)
-							(length 2.54)
-							(name "1"
-								(effects
-									(font
-										(size 1.27 1.27)
-									)
-								)
-							)
-							(number "1"
-								(effects
-									(font
-										(size 1.27 1.27)
-									)
-								)
-							)
-						)
-					)
-					(embedded_fonts no)
-				)
-(version 20250114)
+  (version 20250114)
   (generator "eeschema")
   (generator_version "9.0")
